File: CAN LED Dimmer.kicad_pcb (KiCad board)
At the start: 4 copper layers, 100 x 75 mm, 121 parts, among them IC1 2621011024000, J1 CON_TC2030_SWD, J10 CON_2P_1190297, J2 CON_TC2030_SWD, J3 CON_2P_TBP02R2-381-02BE, J4 CON_2P_TBP02R2-381-02BE, J5 CON_5P_TBP02R2-381-05BE, J6 CON_4P_1190299, J7 CON_2P_1190297, J8 CON_2P_1190297, J9 CON_2P_1190297, Q1 PWR_BTS70202EPAXUMA1, Q10 Q_BSS138_N_CH, Q11 Q_IPD50P04P413ATMA2, Q12 Q_BSS138_N_CH, Q2 PWR_BTS70202EPAXUMA1, Q3 Q_IPD50P04P413ATMA2, Q4 Q_IPD50P04P413ATMA2, Q5 Q_BSS138_N_CH, Q6 Q_IPD50P04P413ATMA2, Q7 Q_IPD90P04P4L04ATMA2, Q8 Q_IPD90P04P4L04ATMA2, Q9 Q_BSS138_N_CH, U1 EEPROM_M24C04-FMC6TG, U2 TLT9251VLEXUMA1, U3 IC_STM32G0B1CCT6, U4 U_LM5166XDRCR, Y1 8MHz

Commit message: optimizing traces
Parts:
- U3: value IC_STM32G0B1CCT6 -> STM32G0B1CEU6; footprint CAN_LED_Dimmer-layout:QFP50P900X900X160-48N_U3 -> CAN_LED_Dimmer-layout:QFN-48-1EP_7x7mm_P0.5mm_EP5.6x5.6mm_U3
Routing:
- net VIN1_ADC: track 60.4 -> 50.1 mm, vias 10 -> 9
- net DEN_A: track 23.7 -> 31.9 mm
- net /MCU - Bluetooth - CAN/BLE_LED1: track 51.4 -> 58.8 mm
- net /MCU - Bluetooth - CAN/BLE_MODE_1: track 25.3 -> 32.5 mm
- net IN0_B: track 68.7 -> 63.0 mm, vias 3 -> 4
- net Net-(U3-PF0): track 26.7 -> 21.0 mm
- net IN0_A: track 63.0 -> 68.6 mm
- net VIN2_ADC: track 43.7 -> 47.9 mm
- net /MCU - Bluetooth - CAN/CAN_RX: track 29.5 -> 26.0 mm
- net /MCU - Bluetooth - CAN/BLE_MODE_0: track 19.3 -> 22.7 mm, vias 2 -> 3
- net /MCU - Bluetooth - CAN/CAN_STBY: track 25.1 -> 27.8 mm
- net /MCU - Bluetooth - CAN/U3_SWDIO: track 32.6 -> 34.7 mm, vias 6 -> 7
- net +3V3: track 202.1 -> 203.9 mm
- net GND: track 16.1 -> 17.4 mm, vias 127 -> 131
- net PWM_0: track 25.7 -> 26.6 mm
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
Commit message: Further layout
Parts:
- I1: value 22uH 2.5A -> 22uH 2.6A; footprint CAN_LED_Dimmer-layout:INDM7166X300N_ASPI-0630LR_I1 -> CAN_LED_Dimmer-layout:SMMS0630-220M_I1
- moved C10 2.44 mm to (163.7, 70.3), turned to -90 degrees
- moved C9 0.67 mm to (162.4, 70.3), turned to -90 degrees
Routing:
- net IN0_A: track 68.6 -> 21.7 mm, vias 9 -> 3
- net /LED Outputs/IS_A: track 21.3 -> 16.7 mm
- net /MCU - Bluetooth - CAN/U3_SWDIO: track 34.7 -> 32.1 mm, vias 7 -> 6
- net +3V3: track 203.9 -> 201.5 mm
- net PWM_3: track 69.2 -> 67.6 mm
- net /MCU - Bluetooth - CAN/DIAG_LED: track 5.76 -> 4.29 mm
- net VIN2_ADC: track 47.9 -> 46.7 mm
- net /MCU - Bluetooth - CAN/CAN_STBY: track 27.8 -> 26.6 mm
- net IN1_A: track 33.0 -> 31.9 mm
- net IN0_B: track 63.0 -> 61.9 mm
- net /MCU - Bluetooth - CAN/BLE_UART_EN: track 35.4 -> 34.5 mm, vias 5 -> 4
- net /MCU - Bluetooth - CAN/BLE_LED1: track 58.8 -> 58.3 mm
- net PWM_1: track 21.8 -> 21.3 mm

Commit message: modified rules
Parts:
- moved D14 11.4 mm to (148.3, 94.7), turned to 180 degrees
- moved C5 10.8 mm to (170.3, 85.9), turned to -90 degrees
- moved C7 8.98 mm to (161.4, 91.0), turned to 90 degrees
- moved R23 8.49 mm to (172.2, 85.2), turned to -90 degrees
- moved U4 6.85 mm to (167.0, 86.9), turned to 180 degrees
- moved R21 5.33 mm to (145.2, 94.4), turned to -90 degrees
- moved B1 3.59 mm to (158.8, 90.3), turned to 0 degrees
- moved I1 3.23 mm to (167.1, 92.4)
- moved C6 2.32 mm to (163.8, 86.8), turned to -90 degrees
- moved F2 1.90 mm to (165.5, 100.4)
- moved U1 1.71 mm to (168.0, 64.3), turned to -90 degrees
- moved C8 1.35 mm to (156.0, 91.1), turned to 90 degrees
Routing:
- net +5V: track 64.5 -> 41.1 mm
- net +3V3: track 201.5 -> 179.4 mm
- net Net-(Q7-G): track 18.8 -> 4.72 mm
- net PWM_2: track 43.8 -> 35.1 mm
- net DEN_B: track 65.1 -> 57.3 mm
- net V_IN_B: track 39.3 -> 47.0 mm
- net GND: track 17.4 -> 13.0 mm, vias 131 -> 134
- net Net-(U4-SW): track 3.95 -> 0.00 mm
- net V_MCU: track 43.7 -> 46.8 mm, vias 3 -> 5
- net IN0_B: track 61.9 -> 59.0 mm
- net IS_A_ADC: track 32.7 -> 29.9 mm
- net Net-(U4-ILIM): track 6.82 -> 4.17 mm
- net DSEL_B: track 58.8 -> 56.7 mm
- net IN1_A: track 31.9 -> 30.6 mm
- net Net-(J6-4.1): track 1.24 -> 0.05 mm
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- added copper zone on F.Cu, net +5V
- added copper zone on F.Cu, net Net-(U4-SW)

Commit message: further layouten
Parts:
- removed UNK_HOLE_0: , CAN_LED_Dimmer-layout:dummyfp0_UNK_HOLE_0
- removed UNK_HOLE_1: , CAN_LED_Dimmer-layout:dummyfp1_UNK_HOLE_1
- removed UNK_HOLE_4: , CAN_LED_Dimmer-layout:dummyfp4_UNK_HOLE_4
- removed UNK_HOLE_5: , CAN_LED_Dimmer-layout:dummyfp5_UNK_HOLE_5
- C3, C4: value 7pF -> 27pF
- C5: value 4.7µF -> 4.7ÂµF
- C6: value 47µF -> 47ÂµF
- C7, C8: value 1µF -> 10µF
- C9: value 1µF -> 1Ã‚ÂµF
- R41: value 4k7 -> 1k; footprint CAN_LED_Dimmer-layout:R_1206_3216Metric_R41 -> CAN_LED_Dimmer-layout:RESC1608X60_R41
- R42: value 4k7 -> 1k; footprint CAN_LED_Dimmer-layout:R_1206_3216Metric_R42 -> CAN_LED_Dimmer-layout:RESC1608X60_R42
- R43: value 4k7 -> 1k; footprint CAN_LED_Dimmer-layout:R_1206_3216Metric_R43 -> CAN_LED_Dimmer-layout:RESC1608X60_R43
- R44: value 4k7 -> 1k; footprint CAN_LED_Dimmer-layout:R_1206_3216Metric_R44 -> CAN_LED_Dimmer-layout:RESC1608X60_R44
- moved D18 61.3 mm to (138.7, 115.8)
- moved R41 58.8 mm to (134.9, 115.9), turned to 0 degrees
- moved D19 49.8 mm to (138.7, 118.4)
- moved R42 46.9 mm to (134.9, 118.6), turned to 0 degrees
- moved D20 39.0 mm to (138.7, 121.0)
- moved R43 35.3 mm to (134.9, 121.3), turned to 0 degrees
- moved D21 29.5 mm to (138.7, 123.6)
- moved R44 24.2 mm to (134.9, 124.0), turned to 0 degrees
- moved C10 13.3 mm to (152.7, 62.9), turned to 0 degrees
- moved C16 13.2 mm to (163.8, 70.3), turned to -90 degrees
- moved C17 12.7 mm to (162.4, 70.3), turned to -90 degrees
- moved C9 11.3 mm to (152.7, 64.5), turned to 0 degrees
- moved R33 5.00 mm to (165.7, 67.7), turned to -90 degrees
- moved R32 4.76 mm to (167.1, 67.7), turned to -90 degrees
- moved C15 3.21 mm to (168.9, 64.2), turned to -90 degrees
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Connections:
- R41 pad 1: /LED Outputs/LED_OUT_1 -> PWM_0
- R42 pad 1: /LED Outputs/LED_OUT_2 -> PWM_1
- R43 pad 1: /LED Outputs/LED_OUT_3 -> PWM_2
- R44 pad 1: /LED Outputs/LED_OUT_4 -> PWM_3
Routing:
- net +3V3: track 179.4 -> 91.2 mm, vias 7 -> 13
- net /MCU - Bluetooth - CAN/U3_SWCLK: track 58.8 -> 20.5 mm, vias 10 -> 4
- net IS_A_ADC: track 29.9 -> 6.75 mm, vias 5 -> 2
- net /MCU - Bluetooth - CAN/U3_RX: track 30.1 -> 13.8 mm, vias 4 -> 2
- net VIN1_ADC: track 50.1 -> 34.4 mm
- net IS_B_ADC: track 64.9 -> 52.9 mm
- net /LED Outputs/LED_OUT_4: track 8.49 -> 0.00 mm
- net /LED Outputs/LED_OUT_3: track 8.49 -> 0.00 mm
- net /LED Outputs/LED_OUT_2: track 8.49 -> 0.00 mm
- net /LED Outputs/LED_OUT_1: track 8.49 -> 0.00 mm
- net Net-(J2-SWDIO/TMS): track 20.3 -> 12.7 mm, vias 4 -> 2
- net /MCU - Bluetooth - CAN/GPIO_BTN3: track 28.6 -> 21.6 mm
- net GND: track 13.0 -> 6.57 mm, vias 134 -> 126
- net Net-(U3-PA2): track 18.2 -> 11.9 mm, vias 4 -> 2
- net IN0_B: track 59.0 -> 53.3 mm
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- added copper zone on In2.Cu, net +3V3
