File: CAN_LED_Dimmer_3.kicad_sch (KiCad schematic)
At the start: 48 parts, among them J10 CON_2P_1190297, J7 CON_2P_1190297, J8 CON_2P_1190297, J9 CON_2P_1190297, Q1 PWR_BTS70202EPAXUMA1, Q10 Q_BSS138_N_CH, Q11 Q_IPD50P04P413ATMA2, Q12 Q_BSS138_N_CH, Q2 PWR_BTS70202EPAXUMA1, Q3 Q_IPD50P04P413ATMA2, Q4 Q_IPD50P04P413ATMA2, Q5 Q_BSS138_N_CH, Q6 Q_IPD50P04P413ATMA2, Q9 Q_BSS138_N_CH

Commit message: modified rules
Parts:
- R41: value 4k7 -> 1k; footprint CAN_LED_Dimmer-layout:R_1206_3216Metric_R41 -> CAN_LED_Dimmer-layout:RESC1608X60_R41; MPN (none) -> RC0603FR-071KL; Power_Rating 0.25 W minimum -> 0.1 W
- R42: value 4k7 -> 1k; footprint CAN_LED_Dimmer-layout:R_1206_3216Metric_R42 -> CAN_LED_Dimmer-layout:RESC1608X60_R42; MPN (none) -> RC0603FR-071KL; Power_Rating 0.25 W minimum -> 0.1 W
- R43: value 4k7 -> 1k; footprint CAN_LED_Dimmer-layout:R_1206_3216Metric_R43 -> CAN_LED_Dimmer-layout:RESC1608X60_R43; MPN (none) -> RC0603FR-071KL; Power_Rating 0.25 W minimum -> 0.1 W
- R44: value 4k7 -> 1k; footprint CAN_LED_Dimmer-layout:R_1206_3216Metric_R44 -> CAN_LED_Dimmer-layout:RESC1608X60_R44; MPN (none) -> RC0603FR-071KL; Power_Rating 0.25 W minimum -> 0.1 W
Connections:
- net LED_OUT_1: no longer R41.1
- net LED_OUT_2: no longer R42.1
- net LED_OUT_3: no longer R43.1
- net LED_OUT_4: no longer R44.1
- net PWM_0: now also R41.1
- net PWM_1: now also R42.1
- net PWM_2: now also R43.1
- net PWM_3: now also R44.1
Other:
- note added: "PWM-Anzeigen: MCU PWM_0..3, 3.3 V, 1k / 0603. Zeigen nur das Steuersignal; keine Ueberwachung der Leistungsausgaenge."
- note removed: "Ausgangsspannungsanzeigen: gruen, 4k7 / 0.25 W, 12 V / 24 V. Helligkeit folgt PWM; keine Laststrom- oder LED-Streifen-Fehlererkennung."
