File: CAN_LED_Dimmer_MCU.kicad_sch (KiCad schematic)
At the start: 44 parts, among them IC1 2621011024000, J1 CON_TC2030_SWD, J2 CON_TC2030_SWD, J3 CON_2P_TBP02R2-381-02BE, J4 CON_2P_TBP02R2-381-02BE, J5 CON_5P_TBP02R2-381-05BE, U1 EEPROM_M24C04-FMC6TG, U2 TLT9251VLEXUMA1, U3 IC_STM32G0B1CCT6, Y1 8MHz

Commit message: optimizing traces
Parts:
- C9: value 1ÂµF -> 1Ã‚ÂµF
- IC1: MANUFACTURER WÃ¼rth Elektronik -> WÃƒÂ¼rth Elektronik
- U3: value IC_STM32G0B1CCT6 -> STM32G0B1CEU6; footprint CAN_LED_Dimmer-layout:QFP50P900X900X160-48N_U3 -> CAN_LED_Dimmer-layout:QFN-48-1EP_7x7mm_P0.5mm_EP5.6x5.6mm_U3; symbol CAN LED Dimmer-eagle-import:IC_STM32G0B1CCT6 -> CAN LED Dimmer-eagle-import:IC_STM32G0B1CEU6; MPN STM32G0B1CCT6 -> STM32G0B1CEU6
Connections:
- net GND: now also U3.49 (VSS)
Changed lines of the file:
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@@
 	)
 	(symbol
-		(lib_id "CAN LED Dimmer-eagle-import:IC_STM32G0B1CCT6")
+		(lib_id "CAN LED Dimmer-eagle-import:IC_STM32G0B1CEU6")
 		(at 208.28 134.62 0)
 		(unit 1)
@@
 			)
 		)
-		(property "Value" "IC_STM32G0B1CCT6"
+		(property "Value" "STM32G0B1CEU6"
 			(at 208.28 149.86 90)
 			(show_name no)
@@
 			)
 		)
-		(property "Footprint" "CAN_LED_Dimmer-layout:QFP50P900X900X160-48N_U3"
+		(property "Footprint" "CAN_LED_Dimmer-layout:QFN-48-1EP_7x7mm_P0.5mm_EP5.6x5.6mm_U3"
 			(at 208.28 134.62 0)
 			(hide yes)
@@
 			)
 		)
-		(property "Datasheet" ""
+		(property "Datasheet" "https://www.st.com/resource/en/datasheet/stm32g0b1ce.pdf"
 			(at 208.28 134.62 0)
 			(hide yes)
@@
 			)
 		)
-		(property "MPN" "STM32G0B1CCT6"
+		(property "MPN" "STM32G0B1CEU6"
 			(at 223.52 148.336 0)
 			(hide yes)
@@
 			)
 		)
-	)
+(pin "49")
+)
 	(symbol
 		(lib_id "CAN LED Dimmer-eagle-import:GND")
@@
 			)
 		)
-		(property "Value" "1ÂµF"
+		(property "Value" "1Ã‚ÂµF"
 			(at 71.12 223.52 0)
 			(show_name no)
@@
 			)
 		)
-		(property "MANUFACTURER" "WÃ¼rth Elektronik"
+		(property "MANUFACTURER" "WÃƒÂ¼rth Elektronik"
 			(at 127 230.124 0)
 			(hide yes)

Commit message: modified rules
Parts:
- C3, C4: value 7pF -> 27pF; MPN (none) -> CL10C270JB8NNNC
- Y1: MPN ABMM-8.000MHZ-D-4-T -> 0175M4-8.000F18DTNJL
